Commit message: Model the real LDROBOT STL-27L LiDAR in sim and training
URDF sensor now matches the D800 kit's STL-27L: 2160 samples/rev, 0.03-25 m,
1.5 cm noise. The policy observation clips ranges to 10 m, the sensor's range on
dark (4%) surfaces, so readings don't depend on wall color. HallwayRaycastEnv
also drops 3% of observed beams during training to mimic missing returns on
glass. Changes the task: models trained before this need retraining.

Co-Authored-By: Claude Opus 5.5 <noreply@anthropic.com>

File: src/cash_sim/urdf/cash_bot.urdf.xacro (robot description, xacro)
@@ -21,5 +21,6 @@
   <xacro:property name="lidar_height" value="0.04"/>
   <xacro:property name="lidar_x"      value="0.05"/>
-  <xacro:property name="lidar_range"  value="12.0"/>
+  <!-- LiDAR: LDROBOT STL-27L (D800 kit); keep the sensor block below in sync with cash_rl/spec.py -->
+  <xacro:property name="lidar_range"  value="25.0"/>
   <!-- ===== Inertia helpers ===== -->
   <xacro:macro name="box_inertia" params="m x y z">
@@ -163,5 +164,5 @@
         <scan>
           <horizontal>
-            <samples>360</samples>
+            <samples>2160</samples>
             <resolution>1</resolution>
             <min_angle>-3.14159</min_angle>
@@ -176,5 +177,5 @@
         </scan>
         <range>
-          <min>0.15</min>
+          <min>0.03</min>
           <max>${lidar_range}</max>
           <resolution>0.01</resolution>
@@ -183,5 +184,5 @@
           <type>gaussian</type>
           <mean>0.0</mean>
-          <stddev>0.01</stddev>
+          <stddev>0.015</stddev>
         </noise>
       </lidar>
